Commit message: simulation: basic movements

File: simulation_ws/src/simulation/robot_description/robot.urdf.xacro (robot description, xacro)
@@ -58,5 +58,5 @@
             <origin xyz="0 ${flip * length/2} 0" rpy="0 0 0"/>
             <axis xyz="0 1 0"/>
-            <limit lower="-2.53073" upper="2.53073" effort="3.8" velocity="60.0"/>
+            <limit lower="-3.14159" upper="3.14159" effort="3.8" velocity="60.0"/>
         </joint>
     </xacro:macro>
@@ -92,5 +92,5 @@
             <origin xyz="0 ${flip * 0.015} -0.175" rpy="0 0 0"/>
             <axis xyz="0 1 0"/>
-            <limit lower="-2.53073" upper="2.53073" effort="3.8" velocity="60.0"/>
+            <limit lower="-3.14159" upper="3.14159" effort="3.8" velocity="60.0"/>
         </joint>
     </xacro:macro>
@@ -117,4 +117,11 @@
                 </geometry>
             </visual>
+            <visual name="${side}_wheel_marker">
+                <origin xyz="0 0 0.06" rpy="0 0 0"/>
+                <geometry><box size="0.02 0.001 0.06"/></geometry>
+                <material name="red">
+                    <color rgba="1 0 0 1"/>
+                </material>
+            </visual>
         </link>
     </xacro:macro>
@@ -127,4 +134,5 @@
             <axis xyz="0 1 0"/>
             <limit effort="3.8" velocity="60.0"/>
+            <dynamics damping="0.005" friction="0"/>
         </joint>
     </xacro:macro>
@@ -150,4 +158,11 @@
             <geometry>
                 <box size="${width} ${length} ${height}"/>
+            </geometry>
+        </visual>
+         <!-- Orientation indicator box -->
+        <visual name='orientation_indicator'>
+            <origin xyz="${width/4} 0 ${height/2 + 0.01}" rpy="0 0 0"/>
+            <geometry>
+                <box size="${width/4} ${length/8} 0.02"/>
             </geometry>
         </visual>
@@ -193,4 +208,5 @@
         <origin xyz="0 0 0.02" rpy="0 0 0"/>
     </joint>
+    <!-- IMU sensor  -->
     <gazebo reference="imu_link">
         <sensor name="imu_sensor" type="imu">
@@ -207,4 +223,5 @@
         </sensor>
     </gazebo>
+    <!-- Gazebo ros_control plugins for the robot -->
     <gazebo>
         <plugin name="gazebo_ros_control" filename="libgazebo_ros_control.so">
@@ -212,4 +229,5 @@
         </plugin>
     </gazebo>
+    <!-- Transmission: turn joints in actuators -->
     <xacro:macro name="transmission" params="joint">
         <transmission name="${joint}_transmission">
@@ -231,3 +249,25 @@
     <xacro:transmission joint="left_wheel_joint"/>
     <xacro:transmission joint="right_wheel_joint"/>
+    <!-- Gazebo friction parameters for the wheels -->
+   <xacro:macro name="friction" params="link">
+  <gazebo reference="${link}">
+    <max_contacts>20</max_contacts>      <!-- keep many points -->
+    <surface>
+      <friction>
+        <ode>
+          <mu>1.0</mu>   <mu2>1.0</mu2>
+          <slip1>0.02</slip1> <slip2>0.02</slip2>   <!-- tiny “give” -->
+        </ode>
+      </friction>
+    </surface>
+  </gazebo>
+</xacro:macro>
+<!--
+<xacro:friction link="left_wheel"/>
+<xacro:friction link="right_wheel"/>
+<xacro:friction link="left_knee"/>
+<xacro:friction link="right_knee"/>
+<xacro:friction link="left_hip"/>
+<xacro:friction link="right_hip"/>
+<xacro:friction link="chassis"/> -->
 </robot>
